Commit message: lab02-gpd: wrist camera URDF, bridge, observation pose, launch fix
- panda_gripper.xacro: add wrist camera link/joint + gz sensor plugin
- gz_bridge.yaml: bridge /wrist_camera/points
- object_detector.py: subscribe to /wrist_camera/points
- grasp_planner_gpd.py: add LOOK_JOINTS + look() + call in main()
- move_group.launch.py: wrap robot_description in ParameterValue

Co-Authored-By: Claude Sonnet 4.6 <noreply@anthropic.com>

File: panda_description/urdf/panda_gripper.xacro (robot description, xacro)
@@ -133,4 +133,46 @@
     gazebo_preserve_fixed_joint="${gazebo_preserve_fixed_joint}"
     />
+    <!-- Wrist camera link: mounted on the back of the hand, looking along the approach axis -->
+    <link name="${prefix}wrist_camera_link"/>
+    <joint name="${prefix}wrist_camera_joint" type="fixed">
+      <parent link="${prefix}${hand_name}"/>
+      <child link="${prefix}wrist_camera_link"/>
+      <!-- 4 cm behind the flange (away from TCP), camera z aligned with hand z (approach dir) -->
+      <origin xyz="0 0 -0.04" rpy="0 0 0"/>
+    </joint>
+    <!-- Gazebo: enable sensor rendering for this model -->
+    <gazebo>
+      <plugin filename="gz-sim-sensors-system" name="gz::sim::systems::Sensors">
+        <render_engine>ogre2</render_engine>
+      </plugin>
+    </gazebo>
+    <!-- Gazebo: RGBD sensor attached to wrist camera link -->
+    <gazebo reference="${prefix}wrist_camera_link">
+      <sensor name="wrist_camera" type="rgbd_camera">
+        <update_rate>10</update_rate>
+        <camera>
+          <horizontal_fov>1.047</horizontal_fov>
+          <image>
+            <width>640</width>
+            <height>480</height>
+            <format>R8G8B8</format>
+          </image>
+          <clip>
+            <near>0.05</near>
+            <far>1.5</far>
+          </clip>
+          <depth_camera>
+            <clip>
+              <near>0.05</near>
+              <far>1.5</far>
+            </clip>
+          </depth_camera>
+        </camera>
+        <always_on>true</always_on>
+        <visualize>true</visualize>
+        <topic>wrist_camera</topic>
+        <gz_frame_id>${prefix}wrist_camera_link</gz_frame_id>
+      </sensor>
+    </gazebo>
     <!-- ROS 2 control -->
     <xacro:if value="${ros2_control}">

Commit message: lab02: clean up skeleton, GPD integration, container setup
- Remove wrist camera from URDF, gz_bridge.yaml, object_detector.py
- Add overhead camera point cloud bridge and static TF in launch
- Add build_transform stub (TODO 2.1) and number all Part 2 TODOs
- Register object_detector.py, grasp_planner.py, grasp_planner_gpd.py in CMakeLists
- Add launch_detector and launch_planner aliases to Dockerfile
- Install libpcl-dev, libopencv-dev, libeigen3-dev and pre-configure GPD cmake
- Fix /ros2_ws → /root/ws paths in LAB02.md bonus section
- Expand alias tables in README.md and LAB02.md

Co-Authored-By: Claude Sonnet 4.6 <noreply@anthropic.com>

File: panda_description/urdf/panda_gripper.xacro (robot description, xacro)
@@ -133,46 +133,4 @@
     gazebo_preserve_fixed_joint="${gazebo_preserve_fixed_joint}"
     />
-    <!-- Wrist camera link: mounted on the back of the hand, looking along the approach axis -->
-    <link name="${prefix}wrist_camera_link"/>
-    <joint name="${prefix}wrist_camera_joint" type="fixed">
-      <parent link="${prefix}${hand_name}"/>
-      <child link="${prefix}wrist_camera_link"/>
-      <!-- 4 cm behind the flange (away from TCP), camera z aligned with hand z (approach dir) -->
-      <origin xyz="0 0 -0.04" rpy="0 0 0"/>
-    </joint>
-    <!-- Gazebo: enable sensor rendering for this model -->
-    <gazebo>
-      <plugin filename="gz-sim-sensors-system" name="gz::sim::systems::Sensors">
-        <render_engine>ogre2</render_engine>
-      </plugin>
-    </gazebo>
-    <!-- Gazebo: RGBD sensor attached to wrist camera link -->
-    <gazebo reference="${prefix}wrist_camera_link">
-      <sensor name="wrist_camera" type="rgbd_camera">
-        <update_rate>10</update_rate>
-        <camera>
-          <horizontal_fov>1.047</horizontal_fov>
-          <image>
-            <width>640</width>
-            <height>480</height>
-            <format>R8G8B8</format>
-          </image>
-          <clip>
-            <near>0.05</near>
-            <far>1.5</far>
-          </clip>
-          <depth_camera>
-            <clip>
-              <near>0.05</near>
-              <far>1.5</far>
-            </clip>
-          </depth_camera>
-        </camera>
-        <always_on>true</always_on>
-        <visualize>true</visualize>
-        <topic>wrist_camera</topic>
-        <gz_frame_id>${prefix}wrist_camera_link</gz_frame_id>
-      </sensor>
-    </gazebo>
     <!-- ROS 2 control -->
     <xacro:if value="${ros2_control}">
